Commit message: Updated Arduino Control Code

File: packages/ros_agv_description/description/robot.urdf.xacro (robot description, xacro)
@@ -2,3 +2,4 @@
 <robot xmlns:xacro="http://www.ros.org/wiki/xacro" name="robot">
     <xacro:include filename="robot_core.xacro" />
+    <xacro:include filename="gazebo_control.xacro" />
 </robot>

File: packages/ros_agv_description/description/robot_core.xacro (robot description, xacro)
@@ -40,4 +40,7 @@
         </xacro:inertial_box>
     </link>
+    <gazebo reference="chassis">
+        <material>Gazebo/White</material>
+    </gazebo>
     <!-- LEFT WHEEL LINK -->
     <joint name="left_wheel_joint" type="continuous">
@@ -63,4 +66,7 @@
         </xacro:inertial_cylinder>
     </link>
+    <gazebo reference="left_wheel">
+        <material>Gazebo/Black</material>
+    </gazebo>
     <!-- RIGHT WHEEL LINK -->
      <joint name="right_wheel_joint" type="continuous">
@@ -86,4 +92,7 @@
         </xacro:inertial_cylinder>
     </link>
+    <gazebo reference="right_wheel">
+        <material>Gazebo/Black</material>
+    </gazebo>
     <!-- Caster-->
     <joint name="caster_joint" type="fixed">
@@ -108,3 +117,8 @@
         </xacro:inertial_sphere>
     </link>
+    <gazebo reference="caster">
+        <material>Gazebo/Black</material>
+        <mu1 value="0.001" />
+        <mu2 value="0.001" />
+    </gazebo>
 </robot>

Commit message: Setup SLAM Toolbox and generated a map

File: packages/ros_agv_description/description/robot.urdf.xacro (robot description, xacro)
@@ -3,3 +3,4 @@
     <xacro:include filename="robot_core.xacro" />
     <xacro:include filename="gazebo_control.xacro" />
+    <xacro:include filename="lidar.xacro" />
 </robot>

File: packages/ros_agv_description/description/robot_core.xacro (robot description, xacro)
@@ -16,4 +16,11 @@
     <!-- BASE LINK -->
     <link name="base_link" />
+    <joint name="base_footprint_joint" type="fixed">
+        <parent link="base_link"/>
+        <child link="base_footprint"/>
+        <origin xyz="0 0 0" rpy="0 0 0" />
+    </joint>
+    <link name="base_footprint">
+    </link>
     <!-- CHASSIS LINK -->
     <joint name="chassis_joint" type="fixed">
